Commit message: Human avatars can be placed with rotation now

File: assets/xacro/human_avatar.xml.xacro (robot description, xacro)
@@ -1,6 +1,6 @@
 <?xml version="1.0"?>
 <mujoco xmlns:xacro="http://ros.org/wiki/xacro">
-<xacro:macro name="human_avatar" params="name pos gesture">
-  <body name="${name}" pos="${pos}">
+<xacro:macro name="human_avatar" params="name pos rot gesture">
+  <body name="${name}" pos="${pos}" euler="${rot}">
     <freejoint/>
     <inertial mass="1" pos="0 0 0" diaginertia="1 1 1"/>

File: scenes/tiago_basic_person.xml.xacro (robot description, xacro)
@@ -34,11 +34,11 @@
   </worldbody>
   <worldbody>
-    <xacro:tiago_robot name="tiago" pos="0 0 0.11" rot="0 0 0" />
+    <xacro:tiago_robot name="tiago" pos="-2 0 0.11" rot="0 0 0" />
   </worldbody>
   <!-- Valid gestures are 'neutral', 'waving_left', 'waving_right', 'pointing_left', 'pointing_right'-->
   <worldbody>
-    <xacro:human_avatar name="human1" pos="1 1 0.95" gesture="waving_left" />
-    <xacro:human_avatar name="human2" pos="-1 1 0.95" gesture="neutral" />
-    <xacro:human_avatar name="human3" pos="1 -1 0.95" gesture="neutral" />
+    <xacro:human_avatar name="human1" pos="0 0 0.95" rot="0 0 3.14" gesture="waving_left" />
+    <xacro:human_avatar name="human2" pos="100 1 0.95" rot="0 0 0" gesture="neutral" />
+    <xacro:human_avatar name="human3" pos="100 -1 0.95" rot="0 0 0" gesture="neutral" />
   </worldbody>
   <xacro:pmb2_contacts name="tiago" />

Commit message: Added postures to avatar. 'standing' and 'sitting' are available for now.

File: assets/xacro/human_avatar.xml.xacro (robot description, xacro)
@@ -1,9 +1,21 @@
 <?xml version="1.0"?>
 <mujoco xmlns:xacro="http://ros.org/wiki/xacro">
-<xacro:macro name="human_avatar" params="name pos rot gesture">
+<!--
+Xacro to generate a human avatar in mujoco. Multiple gestures and postures are available.
+Postures: 'standing', 'sitting'
+Gestures: 'neutral', 'waving_left', 'waving_right', 'pointing_left', 'pointing_right'
+If the avatar is generated sitting, a chair will be placed beneath it.
+-->
+<xacro:macro name="human_avatar" params="name pos rot gesture posture">
   <body name="${name}" pos="${pos}" euler="${rot}">
     <freejoint/>
     <inertial mass="1" pos="0 0 0" diaginertia="1 1 1"/>
     <geom name="${name}_Pelvis" type="mesh" density="0" rgba="0 0 1 1" mesh="Pelvis"/>
+    <!-- Add chair if person is sitting -->
+    <xacro:if value="${posture == 'sitting'}">
+      <body name="${name}_chair">
+          <geom name="${name}_chair" type="cylinder" pos="0 0 -0.33" size="0.2 0.22" rgba=".5 .5 .5 1" />
+      </body>
+    </xacro:if>
     <body name="${name}_LowerTrunk_f1" pos="0 0 0.0663">
       <body name="${name}_LowerTrunk">
@@ -17,4 +29,6 @@
                 <body name="${name}_RightShoulder_f1" pos="0 -0.146767 0">
                   <body name="${name}_RightShoulder_f2">
+                  <!-- Right arm -->
+                  <xacro:unless value="${posture == 'sitting'}">
                     <xacro:if value="${gesture == 'neutral'}">
                       <body name="${name}_RightUpperArm" euler="1.5 0 0">
@@ -32,4 +46,22 @@
                       </body>
                     </xacro:if>
+                  </xacro:unless>
+                  <xacro:if value="${posture == 'sitting'}">
+                    <xacro:if value="${gesture == 'neutral'}">
+                      <body name="${name}_RightUpperArm" euler="1.5 0.2 0.5">
+                        <geom name="${name}_RightUpperArm" pos="0 -0.1581 0" quat="0.707105 0.707108 0 0" type="mesh" density="0" rgba="1 0 0 1" mesh="RightUpperArm"/>
+                        <body name="${name}_RightForeArm_f1" pos="0 -0.3162 0">
+                          <body name="${name}_RightForeArm" euler="0.3 -0.1 0.7">
+                            <geom name="${name}_RightForeArm" pos="0 -0.1241 0" quat="0.707105 0.707108 0 0" type="mesh" density="0" rgba="1 0 0 1" mesh="RightForeArm"/>
+                            <body name="${name}_RightHand_f1" pos="0 -0.2482 0">
+                              <body name="${name}_RightHand" euler="0 1.4 0">
+                                <geom name="${name}_RightHand" pos="0 -0.0718 0" quat="1 0 0 0" type="mesh" density="0" rgba="1 0.76 0.49 1" mesh="RightHand"/>
+                              </body>
+                            </body>
+                          </body>
+                        </body>
+                      </body>
+                    </xacro:if>
+                  </xacro:if>
                     <xacro:if value="${gesture == 'waving_left'}">
                       <body name="${name}_RightUpperArm" euler="1.5 0 0">
@@ -99,4 +131,5 @@
                 <body name="${name}_LeftShoulder_f1" pos="0 0.146767 0">
                   <body name="${name}_LeftShoulder_f2">
+                  <xacro:unless value="${posture == 'sitting'}">
                     <xacro:if value="${gesture == 'neutral'}">
                       <body name="${name}_LeftUpperArm" euler="-1.5 0 0">
@@ -114,4 +147,22 @@
                     </body>
                     </xacro:if>
+                  </xacro:unless>
+                    <xacro:if value="${posture == 'sitting'}">
+                      <xacro:if value="${gesture == 'neutral'}">
+                        <body name="${name}_LeftUpperArm" euler="-1.5 0.2 -0.5">
+                        <geom name="${name}_LeftUpperArm" pos="0 0.1581 0" quat="0.707105 0.707108 0 0" type="mesh" density="0" rgba="1 0 0 1" mesh="LeftUpperArm"/>
+                          <body name="${name}_LeftForeArm_f1" pos="0 0.3162 0">
+                            <body name="${name}_LeftForeArm" euler="-0.3 -0.1 -0.7">
+                              <geom name="${name}_LeftForeArm" pos="0 0.1241 0" quat="0.707105 0.707108 0 0" type="mesh" density="0" rgba="1 0 0 1" mesh="LeftForeArm"/>
+                              <body name="${name}_LeftHand_f1" pos="0 0.2482 0">
+                                <body name="${name}_LeftHand" euler="0 1.4 0">
+                                  <geom name="${name}_LeftHand" pos="0 0.0718 0" quat="1 0 0 0" type="mesh" density="0" rgba="1 0.76 0.49 1" mesh="LeftHand"/>
+                                </body>
+                              </body>
+                            </body>
+                          </body>
+                        </body>
+                      </xacro:if>
+                    </xacro:if>
                     <xacro:if value="${gesture == 'waving_left'}">
                       <body name="${name}_LeftUpperArm" euler="0.75 0 0">
@@ -194,42 +245,88 @@
       </body>
     </body>
-    <body name="${name}_RightUpperLeg_f1" pos="0 -0.09985 -0.0663">
-      <body name="${name}_RightUpperLeg_f2">
-        <body name="${name}_RightUpperLeg">
-          <geom name="${name}_RightUpperLeg" pos="0 0 -0.20825" quat="1 0 0 0" type="mesh" density="0" rgba="0 0 1 1" mesh="RightUpperLeg"/>
-          <body name="${name}_RightLowerLeg_f1" pos="0 0 -0.4165">
-            <body name="${name}_RightLowerLeg">
-              <geom name="${name}_RightLowerLeg" pos="0 0 -0.2091" quat="1 0 0 0" type="mesh" density="0" rgba="0 0 1 1" mesh="RightLowerLeg"/>
-              <body name="${name}_RightFoot_f1" pos="0 0 -0.4182">
-                <body name="${name}_RightFoot_f2">
-                  <body name="${name}_RightFoot">
-                    <geom name="${name}_RightFoot" pos="0.0842 0 -0.03315" quat="1 0 0 0" type="mesh"  density="0" rgba="0.15 0.15 0.15 1" mesh="RightFoot"/>
-                  </body>
-                </body>
-              </body>
-            </body>
-          </body>
-        </body>
-      </body>
-    </body>
-    <body name="${name}_LeftUpperLeg_f1" pos="0 0.09985 -0.0663">
-      <body name="${name}_LeftUpperLeg_f2">
-        <body name="${name}_LeftUpperLeg">
-          <geom name="${name}_LeftUpperLeg" pos="0 0 -0.20825" quat="1 0 0 0" type="mesh" density="0" rgba="0 0 1 1" mesh="LeftUpperLeg"/>
-          <body name="${name}_LeftLowerLeg_f1" pos="0 0 -0.4165">
-            <body name="${name}_LeftLowerLeg">
-              <geom name="${name}_LeftLowerLeg" pos="0 0 -0.2091" quat="1 0 0 0" type="mesh" density="0" rgba="0 0 1 1" mesh="LeftLowerLeg"/>
-              <body name="${name}_LeftFoot_f1" pos="0 0 -0.4182">
-                <body name="${name}_LeftFoot_f2">
-                  <body name="${name}_LeftFoot">
-                    <geom name="${name}_LeftFoot" pos="0.0842 0 -0.03315" quat="1 0 0 0" type="mesh" density="0" rgba="0.15 0.15 0.15 1" mesh="LeftFoot"/>
-                  </body>
-                </body>
-              </body>
-            </body>
-          </body>
-        </body>
-      </body>
-    </body>
+    <xacro:unless value="${posture == 'sitting'}">
+      <body name="${name}_RightUpperLeg_f1" pos="0 -0.09985 -0.0663">
+        <body name="${name}_RightUpperLeg_f2">
+          <body name="${name}_RightUpperLeg">
+            <geom name="${name}_RightUpperLeg" pos="0 0 -0.20825" quat="1 0 0 0" type="mesh" density="0" rgba="0 0 1 1" mesh="RightUpperLeg"/>
+            <body name="${name}_RightLowerLeg_f1" pos="0 0 -0.4165">
+              <body name="${name}_RightLowerLeg">
+                <geom name="${name}_RightLowerLeg" pos="0 0 -0.2091" quat="1 0 0 0" type="mesh" density="0" rgba="0 0 1 1" mesh="RightLowerLeg"/>
+                <body name="${name}_RightFoot_f1" pos="0 0 -0.4182">
+                  <body name="${name}_RightFoot_f2">
+                    <body name="${name}_RightFoot">
+                      <geom name="${name}_RightFoot" pos="0.0842 0 -0.03315" quat="1 0 0 0" type="mesh"  density="0" rgba="0.15 0.15 0.15 1" mesh="RightFoot"/>
+                    </body>
+                  </body>
+                </body>
+              </body>
+            </body>
+          </body>
+        </body>
+      </body>
+    </xacro:unless>
+    <xacro:if value="${posture == 'sitting'}">
+      <body name="${name}_RightUpperLeg_f1" pos="0 -0.09985 -0.0663" euler="0 -1.56 0">
+        <body name="${name}_RightUpperLeg_f2">
+          <body name="${name}_RightUpperLeg">
+            <geom name="${name}_RightUpperLeg" pos="0 0 -0.20825" quat="1 0 0 0" type="mesh" density="0" rgba="0 0 1 1" mesh="RightUpperLeg"/>
+            <body name="${name}_RightLowerLeg_f1" pos="0 0 -0.4165" euler="0 1.56 0">
+              <body name="${name}_RightLowerLeg">
+                <geom name="${name}_RightLowerLeg" pos="0 0 -0.2091" quat="1 0 0 0" type="mesh" density="0" rgba="0 0 1 1" mesh="RightLowerLeg"/>
+                <body name="${name}_RightFoot_f1" pos="0 0 -0.4182">
+                  <body name="${name}_RightFoot_f2">
+                    <body name="${name}_RightFoot">
+                      <geom name="${name}_RightFoot" pos="0.0842 0 -0.03315" quat="1 0 0 0" type="mesh"  density="0" rgba="0.15 0.15 0.15 1" mesh="RightFoot"/>
+                    </body>
+                  </body>
+                </body>
+              </body>
+            </body>
+          </body>
+        </body>
+      </body>
+    </xacro:if>
+    <xacro:unless value="${posture == 'sitting'}">
+      <body name="${name}_LeftUpperLeg_f1" pos="0 0.09985 -0.0663">
+        <body name="${name}_LeftUpperLeg_f2">
+          <body name="${name}_LeftUpperLeg">
+            <geom name="${name}_LeftUpperLeg" pos="0 0 -0.20825" quat="1 0 0 0" type="mesh" density="0" rgba="0 0 1 1" mesh="LeftUpperLeg"/>
+            <body name="${name}_LeftLowerLeg_f1" pos="0 0 -0.4165">
+              <body name="${name}_LeftLowerLeg">
+                <geom name="${name}_LeftLowerLeg" pos="0 0 -0.2091" quat="1 0 0 0" type="mesh" density="0" rgba="0 0 1 1" mesh="LeftLowerLeg"/>
+                <body name="${name}_LeftFoot_f1" pos="0 0 -0.4182">
+                  <body name="${name}_LeftFoot_f2">
+                    <body name="${name}_LeftFoot">
+                      <geom name="${name}_LeftFoot" pos="0.0842 0 -0.03315" quat="1 0 0 0" type="mesh" density="0" rgba="0.15 0.15 0.15 1" mesh="LeftFoot"/>
+                    </body>
+                  </body>
+                </body>
+              </body>
+            </body>
+          </body>
+        </body>
+      </body>
+    </xacro:unless>
+    <xacro:if value="${posture == 'sitting'}">
+      <body name="${name}_LeftUpperLeg_f1" pos="0 0.09985 -0.0663" euler="0 -1.56 0">
+        <body name="${name}_LeftUpperLeg_f2">
+          <body name="${name}_LeftUpperLeg">
+            <geom name="${name}_LeftUpperLeg" pos="0 0 -0.20825" quat="1 0 0 0" type="mesh" density="0" rgba="0 0 1 1" mesh="LeftUpperLeg"/>
+            <body name="${name}_LeftLowerLeg_f1" pos="0 0 -0.4165" euler="0 1.56 0">
+              <body name="${name}_LeftLowerLeg">
+                <geom name="${name}_LeftLowerLeg" pos="0 0 -0.2091" quat="1 0 0 0" type="mesh" density="0" rgba="0 0 1 1" mesh="LeftLowerLeg"/>
+                <body name="${name}_LeftFoot_f1" pos="0 0 -0.4182">
+                  <body name="${name}_LeftFoot_f2">
+                    <body name="${name}_LeftFoot">
+                      <geom name="${name}_LeftFoot" pos="0.0842 0 -0.03315" quat="1 0 0 0" type="mesh" density="0" rgba="0.15 0.15 0.15 1" mesh="LeftFoot"/>
+                    </body>
+                  </body>
+                </body>
+              </body>
+            </body>
+          </body>
+        </body>
+      </body>
+    </xacro:if>
   </body>
 </xacro:macro>
