Commit message: Added ability to spawn human avatar holding pringles in his hand

File: assets/xacro/human_avatar.xml.xacro (robot description, xacro)
@@ -31,5 +31,5 @@
                   <!-- Right arm -->
                   <xacro:unless value="${posture == 'sitting'}">
-                    <xacro:if value="${gesture == 'neutral'}">
+                    <xacro:if value="${gesture == 'neutral' or gesture == 'pointing_left' or gesture == 'waving_left'}">
                       <body name="${name}_RightUpperArm" euler="1.5 0 0">
                         <geom name="${name}_RightUpperArm" pos="0 -0.1581 0" quat="0.707105 0.707108 0 0" type="mesh" density="0" rgba="1 0 0 1" mesh="RightUpperArm"/>
@@ -40,4 +40,23 @@
                               <body name="${name}_RightHand">
                                 <geom name="${name}_RightHand" pos="0 -0.0718 0" quat="1 0 0 0" type="mesh" density="0" rgba="1 0.76 0.49 1" mesh="RightHand"/>
+                              </body>
+                            </body>
+                          </body>
+                        </body>
+                      </body>
+                    </xacro:if>
+                    <xacro:if value="${gesture == 'holding_pringles'}">
+                      <body name="${name}_RightUpperArm" euler="1.5 0.75 0">
+                        <geom name="${name}_RightUpperArm" pos="0 -0.1581 0" quat="0.707105 0.707108 0 0" type="mesh" density="0" rgba="1 0 0 1" mesh="RightUpperArm"/>
+                        <body name="${name}_RightForeArm_f1" pos="0 -0.3162 0" euler="0 0 1.56">
+                          <body name="${name}_RightForeArm">
+                            <geom name="${name}_RightForeArm" pos="0 -0.1241 0" quat="0.707105 0.707108 0 0" type="mesh" density="0" rgba="1 0 0 1" mesh="RightForeArm"/>
+                            <body name="${name}_RightHand_f1" pos="0 -0.2482 0">
+                              <body name="${name}_RightHand">
+                                <geom name="${name}_RightHand" pos="0 -0.0718 0" quat="1 0 0 0" type="mesh" density="0" rgba="1 0.76 0.49 1" mesh="RightHand"/>
+                                <body name="${name}_clf_pringles" pos="0.05 -0.05 -0.045" euler="-1.6 1.55 0">
+                                      <inertial diaginertia="0.005 0.005 0.005" mass="0.05" pos="0 0 0"/>
+                                      <geom name="${name}_clf_pringles" type="mesh" density="0" mesh="clf_Pringles" material="clf_Pringles"/>
+                                </body>
                               </body>
                             </body>
@@ -48,5 +67,5 @@
                   </xacro:unless>
                   <xacro:if value="${posture == 'sitting'}">
-                    <xacro:if value="${gesture == 'neutral'}">
+                    <xacro:if value="${gesture == 'neutral' or gesture == 'pointing_left' or gesture == 'waving_left'}">
                       <body name="${name}_RightUpperArm" euler="1.5 0.2 0.5">
                         <geom name="${name}_RightUpperArm" pos="0 -0.1581 0" quat="0.707105 0.707108 0 0" type="mesh" density="0" rgba="1 0 0 1" mesh="RightUpperArm"/>
@@ -64,19 +83,4 @@
                     </xacro:if>
                   </xacro:if>
-                    <xacro:if value="${gesture == 'waving_left'}">
-                      <body name="${name}_RightUpperArm" euler="1.5 0 0">
-                        <geom name="${name}_RightUpperArm" pos="0 -0.1581 0" quat="0.707105 0.707108 0 0" type="mesh" density="0" rgba="1 0 0 1" mesh="RightUpperArm"/>
-                        <body name="${name}_RightForeArm_f1" pos="0 -0.3162 0">
-                          <body name="${name}_RightForeArm">
-                            <geom name="${name}_RightForeArm" pos="0 -0.1241 0" quat="0.707105 0.707108 0 0" type="mesh" density="0" rgba="1 0 0 1" mesh="RightForeArm"/>
-                            <body name="${name}_RightHand_f1" pos="0 -0.2482 0">
-                              <body name="${name}_RightHand">
-                                <geom name="${name}_RightHand" pos="0 -0.0718 0" quat="1 0 0 0" type="mesh" density="0" rgba="1 0.76 0.49 1" mesh="RightHand"/>
-                              </body>
-                            </body>
-                          </body>
-                        </body>
-                      </body>
-                    </xacro:if>
                     <xacro:if value="${gesture == 'waving_right'}">
                       <body name="${name}_RightUpperArm" euler="-0.75 0 0">
@@ -87,19 +91,4 @@
                             <body name="${name}_RightHand_f1" pos="0 -0.2482 0">
                               <body name="${name}_RightHand" euler="0 -1.5 0">
-                                <geom name="${name}_RightHand" pos="0 -0.0718 0" quat="1 0 0 0" type="mesh" density="0" rgba="1 0.76 0.49 1" mesh="RightHand"/>
-                              </body>
-                            </body>
-                          </body>
-                        </body>
-                      </body>
-                    </xacro:if>
-                    <xacro:if value="${gesture == 'pointing_left'}">
-                      <body name="${name}_RightUpperArm" euler="1.5 0 0">
-                        <geom name="${name}_RightUpperArm" pos="0 -0.1581 0" quat="0.707105 0.707108 0 0" type="mesh" density="0" rgba="1 0 0 1" mesh="RightUpperArm"/>
-                        <body name="${name}_RightForeArm_f1" pos="0 -0.3162 0">
-                          <body name="${name}_RightForeArm">
-                            <geom name="${name}_RightForeArm" pos="0 -0.1241 0" quat="0.707105 0.707108 0 0" type="mesh" density="0" rgba="1 0 0 1" mesh="RightForeArm"/>
-                            <body name="${name}_RightHand_f1" pos="0 -0.2482 0">
-                              <body name="${name}_RightHand">
                                 <geom name="${name}_RightHand" pos="0 -0.0718 0" quat="1 0 0 0" type="mesh" density="0" rgba="1 0.76 0.49 1" mesh="RightHand"/>
                               </body>
@@ -132,5 +121,5 @@
                   <body name="${name}_LeftShoulder_f2">
                   <xacro:unless value="${posture == 'sitting'}">
-                    <xacro:if value="${gesture == 'neutral'}">
+                    <xacro:if value="${gesture == 'neutral' or gesture == 'waving_right' or gesture == 'pointing_right' or gesture == 'holding_pringles'}">
                       <body name="${name}_LeftUpperArm" euler="-1.5 0 0">
                       <geom name="${name}_LeftUpperArm" pos="0 0.1581 0" quat="0.707105 0.707108 0 0" type="mesh" density="0" rgba="1 0 0 1" mesh="LeftUpperArm"/>
@@ -149,5 +138,5 @@
                   </xacro:unless>
                     <xacro:if value="${posture == 'sitting'}">
-                      <xacro:if value="${gesture == 'neutral'}">
+                      <xacro:if value="${gesture == 'neutral' or gesture == 'waving_right' or gesture == 'pointing_right' or gesture == 'holding_pringles'}">
                         <body name="${name}_LeftUpperArm" euler="-1.5 0.2 -0.5">
                         <geom name="${name}_LeftUpperArm" pos="0 0.1581 0" quat="0.707105 0.707108 0 0" type="mesh" density="0" rgba="1 0 0 1" mesh="LeftUpperArm"/>
@@ -180,19 +169,4 @@
                       </body>
                     </xacro:if>
-                    <xacro:if value="${gesture == 'waving_right'}">
-                      <body name="${name}_LeftUpperArm" euler="-1.5 0 0">
-                        <geom name="${name}_LeftUpperArm" pos="0 0.1581 0" quat="0.707105 0.707108 0 0" type="mesh" density="0" rgba="1 0 0 1" mesh="LeftUpperArm"/>
-                        <body name="${name}_LeftForeArm_f1" pos="0 0.3162 0">
-                          <body name="${name}_LeftForeArm">
-                            <geom name="${name}_LeftForeArm" pos="0 0.1241 0" quat="0.707105 0.707108 0 0" type="mesh" density="0" rgba="1 0 0 1" mesh="LeftForeArm"/>
-                            <body name="${name}_LeftHand_f1" pos="0 0.2482 0">
-                              <body name="${name}_LeftHand">
-                                <geom name="${name}_LeftHand" pos="0 0.0718 0" quat="1 0 0 0" type="mesh" density="0" rgba="1 0.76 0.49 1" mesh="LeftHand"/>
-                              </body>
-                            </body>
-                          </body>
-                        </body>
-                      </body>
-                    </xacro:if>
                     <xacro:if value="${gesture == 'pointing_left'}">
                       <body name="${name}_LeftUpperArm" euler="-0.5 0 0">
@@ -203,19 +177,4 @@
                             <body name="${name}_LeftHand_f1" pos="0 0.2482 0">
                               <body name="${name}_LeftHand" euler="0 -1.5 0">
-                                <geom name="${name}_LeftHand" pos="0 0.0718 0" quat="1 0 0 0" type="mesh" density="0" rgba="1 0.76 0.49 1" mesh="LeftHand"/>
-                              </body>
-                            </body>
-                          </body>
-                        </body>
-                      </body>
-                    </xacro:if>
-                    <xacro:if value="${gesture == 'pointing_right'}">
-                      <body name="${name}_LeftUpperArm" euler="-1.5 0 0">
-                        <geom name="${name}_LeftUpperArm" pos="0 0.1581 0" quat="0.707105 0.707108 0 0" type="mesh" density="0" rgba="1 0 0 1" mesh="LeftUpperArm"/>
-                        <body name="${name}_LeftForeArm_f1" pos="0 0.3162 0">
-                          <body name="${name}_LeftForeArm">
-                            <geom name="${name}_LeftForeArm" pos="0 0.1241 0" quat="0.707105 0.707108 0 0" type="mesh" density="0" rgba="1 0 0 1" mesh="LeftForeArm"/>
-                            <body name="${name}_LeftHand_f1" pos="0 0.2482 0">
-                              <body name="${name}_LeftHand">
                                 <geom name="${name}_LeftHand" pos="0 0.0718 0" quat="1 0 0 0" type="mesh" density="0" rgba="1 0.76 0.49 1" mesh="LeftHand"/>
                               </body>

File: scenes/tiago_basic_person.xml.xacro (robot description, xacro)
@@ -36,5 +36,5 @@
     <xacro:tiago_robot name="tiago" pos="-2 0 0.11" rot="0 0 0" />
   </worldbody>
-  <!-- Valid gestures are 'neutral', 'waving_left', 'waving_right', 'pointing_left', 'pointing_right'-->
+  <!-- Valid gestures are 'neutral', 'waving_left', 'waving_right', 'pointing_left', 'pointing_right', 'holding_pringles'-->
   <!-- Valid postures are 'standing', 'sitting'-->
   <worldbody>
@@ -42,6 +42,4 @@
     <xacro:human_avatar name="human2" pos="100 1 0.95" rot="0 0 0" gesture="neutral" posture="standing" />
     <xacro:human_avatar name="human3" pos="100 -1 0.95" rot="0 0 0" gesture="neutral" posture="standing" />
-    <xacro:human_avatar name="human4" pos="1 1 0.55" rot="0 0 0" gesture="neutral" posture="sitting" />
-    <xacro:human_avatar name="human5" pos="2 2 0.55" rot="0 0 0" gesture="waving_left" posture="sitting" />
   </worldbody>
   <xacro:pmb2_contacts name="tiago" />
