Commit message: Added pos support to macro

File: model_makros/clf/couch_office_table_2m.xml.xacro (robot description, xacro)
@@ -1,5 +1,5 @@
 <?xml version="1.0" ?>
 <mujoco xmlns:xacro="http://ros.org/wiki/xacro">
-  <xacro:macro name="add_office_table_2m" params="geom_name pos:='0 0 0'">
+  <xacro:macro name="add_couch_office_table_2m" params="geom_name pos:='0 0 0'">
     <worldbody>
       <body name="${geom_name}_body" pos="${pos}">

File: model_makros/clf/couch_table.xml.xacro (robot description, xacro)
@@ -1,7 +1,7 @@
 <?xml version="1.0" ?>
 <mujoco xmlns:xacro="http://ros.org/wiki/xacro">
-  <xacro:macro name="add_couch_table" params="geom_name">
+  <xacro:macro name="add_couch_table" params="geom_name pos:='0 0 0'">
     <worldbody>
-      <body name="${geom_name}_body">
+      <body name="${geom_name}_body" pos="${pos}">
         <geom name="${geom_name}_box_0" type="box" pos="0.0 0.0 0.425" size="0.45 0.275 0.02525" rgba="0.5 0.5 0.5 1" density="1000"/>
         <geom name="${geom_name}_box_1" type="box" pos="0.0 0.0 0.205" size="0.45 0.225 0.005" rgba="0.5 0.5 0.5 1" density="1000"/>

File: model_makros/clf/ikea_table.xml.xacro (robot description, xacro)
@@ -1,7 +1,7 @@
 <?xml version="1.0" ?>
 <mujoco xmlns:xacro="http://ros.org/wiki/xacro">
-  <xacro:macro name="add_ikea_table" params="geom_name">
+  <xacro:macro name="add_ikea_table" params="geom_name pos:='0 0 0'">
     <worldbody>
-      <body name="${geom_name}_body">
+      <body name="${geom_name}_body" pos="${pos}">
         <geom name="${geom_name}_box_0" type="box" pos="0.0 0.0 0.7415" size="0.4 0.6 0.0085" rgba="0.5 0.5 0.5 1" density="1000"/>
         <geom name="${geom_name}_box_1" type="box" pos="-0.38 -0.58 0.366" size="0.02 0.02 0.366" rgba="0.5 0.5 0.5 1" density="1000"/>

File: model_makros/clf/office_table_1m.xml.xacro (robot description, xacro)
@@ -1,7 +1,7 @@
 <?xml version="1.0" ?>
 <mujoco xmlns:xacro="http://ros.org/wiki/xacro">
-  <xacro:macro name="add_office_table_1m" params="geom_name">
+  <xacro:macro name="add_office_table_1m" params="geom_name pos:='0 0 0'">
     <worldbody>
-      <body name="${geom_name}_body">
+      <body name="${geom_name}_body" pos="${pos}">
         <geom name="${geom_name}_box_0" type="box" pos="0.0 0.0 0.7075" size="0.4 0.5 0.0125" rgba="0.5 0.5 0.5 1" density="1000"/>
         <geom name="${geom_name}_box_1" type="box" pos="0.375 0.455 0.3475" size="0.0155 0.0155 0.3475" rgba="0.5 0.5 0.5 1" density="1000"/>

File: model_makros/clf/office_table_1m20.xml.xacro (robot description, xacro)
@@ -1,7 +1,7 @@
 <?xml version="1.0" ?>
 <mujoco xmlns:xacro="http://ros.org/wiki/xacro">
-  <xacro:macro name="add_office_table_1m20" params="geom_name">
+  <xacro:macro name="add_office_table_1m20" params="geom_name pos:='0 0 0'">
     <worldbody>
-      <body name="${geom_name}_body">
+      <body name="${geom_name}_body" pos="${pos}">
         <geom name="${geom_name}_box_0" type="box" pos="0.0 0.0 0.7075" size="0.4 0.6 0.0125" rgba="0.5 0.5 0.5 1" density="1000"/>
         <geom name="${geom_name}_box_1" type="box" pos="0.375 0.555 0.3475" size="0.0155 0.0155 0.3475" rgba="0.5 0.5 0.5 1" density="1000"/>

File: model_makros/clf/office_table_1m40.xml.xacro (robot description, xacro)
@@ -1,7 +1,7 @@
 <?xml version="1.0" ?>
 <mujoco xmlns:xacro="http://ros.org/wiki/xacro">
-  <xacro:macro name="add_office_table_1m40" params="geom_name">
+  <xacro:macro name="add_office_table_1m40" params="geom_name pos:='0 0 0'">
     <worldbody>
-      <body name="${geom_name}_body">
+      <body name="${geom_name}_body" pos="${pos}">
         <geom name="${geom_name}_box_0" type="box" pos="0.0 0.0 0.7075" size="0.3 0.7 0.0125" rgba="0.5 0.5 0.5 1" density="1000"/>
         <geom name="${geom_name}_box_1" type="box" pos="0.275 0.655 0.3475" size="0.0155 0.0155 0.3475" rgba="0.5 0.5 0.5 1" density="1000"/>

File: model_makros/clf/office_table_1m60.xml.xacro (robot description, xacro)
@@ -1,7 +1,7 @@
 <?xml version="1.0" ?>
 <mujoco xmlns:xacro="http://ros.org/wiki/xacro">
-  <xacro:macro name="add_office_table_1m60" params="geom_name">
+  <xacro:macro name="add_office_table_1m60" params="geom_name pos:='0 0 0'">
     <worldbody>
-      <body name="${geom_name}_body">
+      <body name="${geom_name}_body" pos="${pos}">
         <geom name="${geom_name}_box_0" type="box" pos="0.0 0.0 0.7075" size="0.4 0.8 0.0125" rgba="0.5 0.5 0.5 1" density="1000"/>
         <geom name="${geom_name}_box_1" type="box" pos="0.375 0.755 0.3475" size="0.0155 0.0155 0.3475" rgba="0.5 0.5 0.5 1" density="1000"/>

File: model_makros/clf/office_table_1m80.xml.xacro (robot description, xacro)
@@ -1,7 +1,7 @@
 <?xml version="1.0" ?>
 <mujoco xmlns:xacro="http://ros.org/wiki/xacro">
-  <xacro:macro name="add_office_table_1m80" params="geom_name">
+  <xacro:macro name="add_office_table_1m80" params="geom_name pos:='0 0 0'">
     <worldbody>
-      <body name="${geom_name}_body">
+      <body name="${geom_name}_body" pos="${pos}">
         <geom name="${geom_name}_box_0" type="box" pos="0.0 0.0 0.7075" size="0.4 0.9 0.0125" rgba="0.5 0.5 0.5 1" density="1000"/>
         <geom name="${geom_name}_box_1" type="box" pos="0.375 0.855 0.3475" size="0.0155 0.0155 0.3475" rgba="0.5 0.5 0.5 1" density="1000"/>

File: model_makros/clf/red_billy.xml.xacro (robot description, xacro)
@@ -1,7 +1,7 @@
 <?xml version="1.0" ?>
 <mujoco xmlns:xacro="http://ros.org/wiki/xacro">
-  <xacro:macro name="add_red_billy" params="geom_name">
+  <xacro:macro name="add_red_billy" params="geom_name pos:='0 0 0'">
     <worldbody>
-      <body name="${geom_name}_body">
+      <body name="${geom_name}_body" pos="${pos}">
         <geom name="${geom_name}_box_0" type="box" pos="-0.39 0.0 1.01" size="0.01 0.14 1.01" rgba="0.5 0.5 0.5 1" density="1000"/>
         <geom name="${geom_name}_box_1" type="box" pos="0.39 0.0 1.01" size="0.01 0.14 1.01" rgba="0.5 0.5 0.5 1" density="1000"/>
