Commit message: Added covers to generated models. Added scene for challenge ws25.

File: model_makros/clf/covered/couch_table.xml.xacro (robot description, xacro)
@@ -10,4 +10,5 @@
         <geom name="${geom_name}_box_4" type="box" pos="0.425 -0.25 0.2" size="0.025 0.025 0.2" rgba="0.5 0.5 0.5 1" density="1000"/>
         <geom name="${geom_name}_box_5" type="box" pos="-0.425 -0.25 0.2" size="0.025 0.025 0.2" rgba="0.5 0.5 0.5 1" density="1000"/>
+        <geom name="${geom_name}_box_cover" type="box" pos="0.0 0.0 0.05" size="0.45 0.275 0.05" rgba="0.73 0.82 1 0.8" density="1000"/>
       </body>
     </worldbody>

File: model_makros/clf/covered/ikea_table.xml.xacro (robot description, xacro)
@@ -9,4 +9,5 @@
         <geom name="${geom_name}_box_3" type="box" pos="-0.38 0.58 0.366" size="0.02 0.02 0.366" rgba="0.5 0.5 0.5 1" density="1000"/>
         <geom name="${geom_name}_box_4" type="box" pos="0.38 0.58 0.366" size="0.02 0.02 0.366" rgba="0.5 0.5 0.5 1" density="1000"/>
+        <geom name="${geom_name}_box_cover" type="box" pos="0.0 0.0 0.05" size="0.4 0.6 0.05" rgba="0.73 0.82 1 0.8" density="1000"/>
       </body>
     </worldbody>

File: model_makros/clf/covered/office_table_2m.xml.xacro (robot description, xacro)
@@ -1,7 +1,7 @@
 <?xml version="1.0" ?>
 <mujoco xmlns:xacro="http://ros.org/wiki/xacro">
-  <xacro:macro name="add_couch_office_table_2m" params="geom_name pos:='0 0 0'">
+  <xacro:macro name="add_office_table_2m" params="geom_name pos:='0 0 0' rot:='0 0 0'">
     <worldbody>
-      <body name="${geom_name}_body" pos="${pos}">
+      <body name="${geom_name}_body" pos="${pos}" euler="${rot}">
         <geom name="${geom_name}_box_0" type="box" pos="0.0 0.0 0.7075" size="0.4 1.0 0.0125" rgba="0.5 0.5 0.5 1" density="1000"/>
         <geom name="${geom_name}_box_1" type="box" pos="0.375 0.955 0.3475" size="0.0155 0.0155 0.3475" rgba="0.5 0.5 0.5 1" density="1000"/>
@@ -9,4 +9,5 @@
         <geom name="${geom_name}_box_3" type="box" pos="0.375 -0.955 0.3475" size="0.0155 0.0155 0.3475" rgba="0.5 0.5 0.5 1" density="1000"/>
         <geom name="${geom_name}_box_4" type="box" pos="-0.375 -0.955 0.3475" size="0.0155 0.0155 0.3475" rgba="0.5 0.5 0.5 1" density="1000"/>
+        <geom name="${geom_name}_box_cover" type="box" pos="0.0 0.0 0.05" size="0.4 1.0 0.05" rgba="0.73 0.82 1 0.8" density="1000"/>
       </body>
     </worldbody>

File: model_makros/clf/covered/red_billy.xml.xacro (robot description, xacro)
@@ -14,4 +14,5 @@
         <geom name="${geom_name}_box_8" type="box" pos="0.0 0.01 1.42" size="0.38 0.13 0.01" rgba="0.5 0.5 0.5 1" density="1000"/>
         <geom name="${geom_name}_box_9" type="box" pos="0.0 0.01 1.805" size="0.38 0.13 0.01" rgba="0.5 0.5 0.5 1" density="1000"/>
+        <geom name="${geom_name}_box_cover" type="box" pos="0.0 0.0 0.05" size="0.4 0.14 0.05" rgba="0.73 0.82 1 0.8" density="1000"/>
       </body>
     </worldbody>

File: model_makros/clf/office_table_2m.xml.xacro (robot description, xacro)
@@ -1,7 +1,7 @@
 <?xml version="1.0" ?>
 <mujoco xmlns:xacro="http://ros.org/wiki/xacro">
-  <xacro:macro name="add_office_table_2m" params="geom_name pos:='0 0 0'">
+  <xacro:macro name="add_office_table_2m" params="geom_name pos:='0 0 0' rot:='0 0 0'">
     <worldbody>
-      <body name="${geom_name}_body" pos="${pos}">
+      <body name="${geom_name}_body" pos="${pos}" euler="${rot}">
         <geom name="${geom_name}_box_0" type="box" pos="0.0 0.0 0.7075" size="0.4 1.0 0.0125" rgba="0.5 0.5 0.5 1" density="1000"/>
         <geom name="${geom_name}_box_1" type="box" pos="0.375 0.955 0.3475" size="0.0155 0.0155 0.3475" rgba="0.5 0.5 0.5 1" density="1000"/>
@@ -9,4 +9,5 @@
         <geom name="${geom_name}_box_3" type="box" pos="0.375 -0.955 0.3475" size="0.0155 0.0155 0.3475" rgba="0.5 0.5 0.5 1" density="1000"/>
         <geom name="${geom_name}_box_4" type="box" pos="-0.375 -0.955 0.3475" size="0.0155 0.0155 0.3475" rgba="0.5 0.5 0.5 1" density="1000"/>
+        <geom name="${geom_name}_box_cover" type="box" pos="0.0 0.0 0.04" size="0.4 1.0 0.04" rgba="0.73 0.82 1 0.8" density="1000"/>
       </body>
     </worldbody>
