Commit message: Added furniture to cologne scene

File: scenes/cologne2026.xml.xacro (robot description, xacro)
@@ -73,116 +73,177 @@
 		<mesh name="misc/seating" file="$(find ecwm_data)/models/misc/seating/meshes/textured.stl" />
 	</asset>
+	<contact>
+		<exclude body1="dishwasher" body2="dishwasher_door" />
+		<exclude body1="dishwasher" body2="dishwasher_drawer_lower" />
+		<exclude body1="dishwasher" body2="dishwasher_drawer_upper" />
+	</contact>
+	<asset />
 	<worldbody>
-		<body name="working_table2" pos="7.794271469116211 -4.350337028503418 3.725290298461914e-09"
-			quat="0.001113440698489049 -4.750988378298072e-10 -5.291750800243135e-10 -0.9999993801247133">
-			<geom type="box" size="0.035 0.035 0.35" pos="-0.965 -0.365 0.3475" quat="1 0 0 0" />
-			<geom type="box" size="0.035 0.035 0.35" pos="0.965 -0.365 0.3475" quat="1 0 0 0" />
-			<geom type="box" size="0.035 0.035 0.35" pos="-0.965 0.365 0.3475" quat="1 0 0 0" />
-			<geom type="box" size="0.035 0.035 0.35" pos="0.965 0.365 0.3475" quat="1 0 0 0" />
-			<geom type="box" size="1 0.4 0.0105" pos="0 0 0.7075" quat="1 0 0 0" />
-		</body>
-		<body name="working_table1" pos="5.793829441070557 -4.355586051940918 9.238719940185547e-07"
-			quat="0.999956534118101 -2.6423678872177553e-08 -1.8286666145577964e-08 -0.009323619174657372">
-			<geom type="box" size="0.035 0.035 0.35" pos="-0.944 -0.365 0.3475" quat="1 0 0 0" />
-			<geom type="box" size="0.035 0.035 0.35" pos="0.944 -0.365 0.3475" quat="1 0 0 0" />
-			<geom type="box" size="0.035 0.035 0.35" pos="-0.944 0.365 0.3475" quat="1 0 0 0" />
-			<geom type="box" size="0.035 0.035 0.35" pos="0.944 0.365 0.3475" quat="1 0 0 0" />
-			<geom type="box" size="0.979 0.4 0.0105" pos="0 0 0.7075" quat="1 0 0 0" />
-		</body>
-		<body name="trashbin" pos="3.774446964263916 2.558544874191284 0"
+		<body name="washingmaschine" pos="5.658462047576904 -0.971213698387146 0"
+			quat="-0.02897400681516465 4.0457522220899846e-10 1.3402909679074348e-09 0.999580165333964">
+			<geom type="box" size="0.3 0.3 0.425" pos="0 0 0.425" quat="1 0 0 0" />
+		</body>
+		<body name="wall_4" pos="6.104307651519775 -0.8419799208641052 3.3527612686157227e-07"
+			quat="0.9995062151309462 -2.41655490780669e-08 -1.100961344497049e-08 0.03142174270485421">
+			<geom type="box" size="0.05 0.4 1" pos="-0.05 0 1" quat="1 0 0 0" />
+		</body>
+		<body name="wall_3" pos="6.152462005615234 -1.6543262004852295 7.338821887969971e-07"
+			quat="0.9997148048534122 -2.30484726816154e-08 -1.1270307933929542e-08 0.023881142286400186">
+			<geom type="box" size="0.05 0.4 1" pos="-0.05 0 1" quat="1 0 0 0" />
+		</body>
+		<body name="wall_2" pos="8.53603458404541 -1.860910415649414 1.5869736671447754e-06"
+			quat="0.6962954881211747 -5.1075384841798485e-08 -2.3256519875004202e-08 0.7177552460428918">
+			<geom type="box" size="0.05 0.4 1" pos="-0.05 0 1" quat="1 0 0 0" />
+		</body>
+		<body name="wall_1" pos="6.535908222198486 -1.9599981307983398 1.257285475730896e-06"
+			quat="0.6845936263344012 -5.1444005244362393e-08 -2.3416341154278974e-08 0.7289249390590988">
+			<geom type="box" size="0.05 0.4 1" pos="-0.05 0 1" quat="1 0 0 0" />
+		</body>
+		<body name="tv_stand" pos="4.885616779327393 6.018153667449951 0"
+			quat="-0.026212220312108236 -8.417049870878699e-13 1.5637258847026423e-09 0.9996564007229233">
+			<geom type="box" size="0.03 0.37 0.2425" pos="0 0 0.6075" quat="1 0 0 0" />
+			<geom type="box" size="0.1735 0.76 0.1825" pos="0 0 0.1825" quat="1 0 0 0" />
+		</body>
+		<body name="trash_bin" pos="6.596708297729492 -1.6754956245422363 1.8998980522155762e-07"
 			quat="0.9998455855472655 -1.4333701708010158e-08 -3.448968328074148e-09 -0.01757285012869549">
 			<geom type="box" size="0.025 0.025 0.025" pos="0 0 0.025" quat="1 0 0 0" />
 		</body>
-		<body name="stool2" pos="6.0038580894470215 -0.3694360554218292 2.384185791015625e-07"
-			quat="0.0019943099036485567 6.453821781376714e-10 -1.6989687066270616e-10 -0.9999980113620268">
-			<geom type="box" size="0.25 0.2075 0.225" pos="0 0 0.225" quat="1 0 0 0" />
-		</body>
-		<body name="stool1" pos="4.594932556152344 -2.484583854675293 8.791685104370117e-07"
-			quat="-0.0020146665570880133 -2.885629149520463e-08 3.026432429260701e-08 0.9999979705572718">
-			<geom type="box" size="0.25 0.2075 0.225" pos="0 0 0.225" quat="1 0 0 0" />
-		</body>
-		<body name="shelf" pos="4.427527904510498 3.0427048206329346 1.844950020313263e-06"
-			quat="-0.002034059053080725 8.136556910808678e-08 -1.513866211567279e-08 -0.9999979312997411">
-			<geom type="box" size="0.38 0.133 0.01" pos="0 0.007000000000000006 1.9960000000000002"
-				quat="1 0 0 0" />
-			<geom type="box" size="0.38 0.133 0.01" pos="0 0.007000000000000006 1.7730000000000001"
-				quat="1 0 0 0" />
-			<geom type="box" size="0.38 0.133 0.01" pos="0 0.007000000000000006 1.3880000000000001"
-				quat="1 0 0 0" />
-			<geom type="box" size="0.38 0.133 0.01" pos="0 0.007000000000000006 1.0339999999999998"
-				quat="1 0 0 0" />
-			<geom type="box" size="0.38 0.133 0.01" pos="0 0.007000000000000006 0.743"
-				quat="1 0 0 0" />
-			<geom type="box" size="0.38 0.133 0.01" pos="0 0.007000000000000006 0.39" quat="1 0 0 0" />
-			<geom type="box" size="0.38 0.133 0.01" pos="0 0.007000000000000006 0.07" quat="1 0 0 0" />
-			<geom type="box" size="0.38 0.007000000000000006 1.01" pos="0 -0.133 1.01"
+		<body name="sink" pos="7.65725564956665 -1.6599617004394531 0"
+			quat="0.6868477137209862 0 0 0.7268013608657142">
+			<geom type="box" size="0.215 0.6 0.1715" pos="-0.1275 0 1.7215" quat="1 0 0 0" />
+			<geom type="box" size="0.14 0.6 0.25" pos="-0.2025 0 1.3" quat="1 0 0 0" />
+			<geom type="box" size="0.3425 0.3 0.525" pos="0 -0.3 0.5025" quat="1 0 0 0" />
+		</body>
+		<body name="shelf" pos="5.284006118774414 2.102001667022705 9.872019290924072e-07"
+			quat="0.9995322484121183 -6.764413950953164e-10 -6.135356181776e-08 0.030582419528409753">
+			<geom type="box" size="0.38 0.1325 0.01" pos="0 0.007500000000000007 2.007"
+				quat="1 0 0 0" />
+			<geom type="box" size="0.38 0.1325 0.01" pos="0 0.007500000000000007 1.429"
+				quat="1 0 0 0" />
+			<geom type="box" size="0.38 0.1325 0.01" pos="0 0.007500000000000007 1.049"
+				quat="1 0 0 0" />
+			<geom type="box" size="0.38 0.1325 0.01" pos="0 0.007500000000000007 0.759"
+				quat="1 0 0 0" />
+			<geom type="box" size="0.38 0.1325 0.01"
+				pos="0 0.007500000000000007 0.44000000000000006" quat="1 0 0 0" />
+			<geom type="box" size="0.38 0.1325 0.01"
+				pos="0 0.007500000000000007 0.09000000000000001" quat="1 0 0 0" />
+			<geom type="box" size="0.38 0.007500000000000007 1.01" pos="0 -0.1325 1.01"
 				quat="1 0 0 0" />
 			<geom type="box" size="0.01 0.14 1.01" pos="0.39 0 1.01" quat="1 0 0 0" />
 			<geom type="box" size="0.01 0.14 1.01" pos="-0.39 0 1.01" quat="1 0 0 0" />
 		</body>
-		<body name="seat_4" pos="7.131048202514648 1.6653859615325928 1.0952353477478027e-06"
-			quat="0.6965711463598729 -9.8445237769765e-08 -9.281268754523073e-09 0.7174877267653313">
-			<geom type="mesh" mesh="misc/seating_COLLISION" group="3" />
-			<geom type="mesh" mesh="misc/seating" material="misc/seating" contype="0"
-				conaffinity="0" group="2" />
-		</body>
-		<body name="seat_3" pos="7.311963081359863 -3.444875955581665 1.6167759895324707e-06"
-			quat="0.9507858688617007 -2.3136838065911566e-08 -5.457251680117766e-08 0.3098487236909287">
-			<geom type="mesh" mesh="misc/seating_COLLISION" group="3" />
-			<geom type="mesh" mesh="misc/seating" material="misc/seating" contype="0"
-				conaffinity="0" group="2" />
-		</body>
-		<body name="seat_2" pos="5.500264644622803 1.7026004791259766 1.4901161193847656e-08"
-			quat="0.7209090152580562 4.036902833275319e-08 3.4058327421214546e-09 -0.6930297192182008">
-			<geom type="mesh" mesh="misc/seating_COLLISION" group="3" />
-			<geom type="mesh" mesh="misc/seating" material="misc/seating" contype="0"
-				conaffinity="0" group="2" />
-		</body>
-		<body name="seat_1" pos="7.092272758483887 -1.2040947675704956 1.4901161193847656e-08"
-			quat="0.20447152332916366 7.509208064202577e-10 -1.2213007183559397e-08 0.9788725127142203">
-			<geom type="mesh" mesh="misc/seating_COLLISION" group="3" />
-			<geom type="mesh" mesh="misc/seating" material="misc/seating" contype="0"
-				conaffinity="0" group="2" />
-		</body>
-		<body name="round_table" pos="7.359313011169434 0.09826286882162094 1.601874828338623e-07"
-			quat="0.7083268769037853 1.6348411530520224e-10 -4.067501548165117e-11 -0.7058845765815611">
+		<body name="night_stand" pos="4.260159492492676 4.56071662902832 0"
+			quat="-0.015960043384359895 1.4529149665069498e-11 9.834614288407655e-10 0.9998726303960767">
+			<geom type="box" size="0.25 0.25 0.25" pos="0 0 0.25" quat="1 0 0 0" />
+		</body>
+		<body name="kitchen_counter" pos="6.916921138763428 1.4336552619934082 0"
+			quat="0.6906426435978936 -2.2696938401593248e-10 9.100149373957736e-10 0.7231961966466036">
+			<geom type="box" size="0.5 0.5 0.5" pos="0 0 0.5" quat="1 0 0 0" />
+		</body>
+		<body name="garbage_bin" pos="4.960423469543457 4.344700336456299 0"
+			quat="0.9998455855472655 -1.4333701708010158e-08 -3.448968328074148e-09 -0.01757285012869549">
+			<geom type="box" size="0.025 0.025 0.025" pos="0 0 0.025" quat="1 0 0 0" />
+		</body>
+		<body name="fridge" pos="7.662601470947266 -1.6627413034439087 0"
+			quat="0.6868477137209862 0 0 0.7268013608657142">
+			<geom type="box" size="0.3425 0.3 0.525" pos="0 0.3 0.5025" quat="1 0 0 0" />
+		</body>
+		<body name="dresser" pos="0.9144766926765442 4.809781074523926 0"
+			quat="-0.04235903833446693 -8.332604577297311e-11 2.5689072573684127e-09 0.9991024531405072">
+			<geom type="box" size="0.1515 0.31 0.3475" pos="0 0 0.3475" quat="1 0 0 0" />
+		</body>
+		<body name="drawer" pos="6.053994178771973 7.8024821281433105 0"
+			quat="-0.008640857237164429 -5.687957974622105e-11 2.9145998908278466e-10 0.9999626670962307">
+			<geom type="box" size="0.17 0.15 0.28" pos="0 0 0.28" quat="1 0 0 0" />
+		</body>
+		<body name="dishwasher" pos="8.555129051208496 -1.562673807144165 0"
+			quat="0.9996288385807544 -1.8498175152824488e-09 1.6130728644026446e-10 0.027243073939851304">
+			<body name="dishwasher_door" pos="0 0.26 0.15" quat="0 0 0 1">
+				<geom type="box" size="0.025 0.025 0.025" pos="0 0 0" quat="1 0 0 0" />
+				<geom type="box" size="0.3 0.025 0.362" pos="0 0 0.2975" quat="1 0 0 0" />
+				<joint type="hinge" axis="0 1 0" range="0 1.57" />
+			</body>
+			<body name="dishwasher_drawer_lower" pos="0 -0.05 0.24" quat="1 0 0 0">
+				<geom type="box" size="0.01 0.125 0.1" pos="0 0.085 0.1" quat="1 0 0 0" />
+				<geom type="box" size="0.005 0.26 0.05" pos="-0.2575 0 0.05" quat="1 0 0 0" />
+				<geom type="box" size="0.005 0.26 0.05" pos="0.2575 0 0.05" quat="1 0 0 0" />
+				<geom type="box" size="0.2625 0.005 0.05" pos="0 -0.255 0.05" quat="1 0 0 0" />
+				<geom type="box" size="0.2625 0.005 0.05" pos="0 0.255 0.05" quat="1 0 0 0" />
+				<geom type="box" size="0.2625 0.26 0.005" pos="0 0 0.005" quat="1 0 0 0" />
+				<joint type="slide" axis="0 1 0" range="0 0.54" />
+			</body>
+			<body name="dishwasher_drawer_upper" pos="0 -0.05 0.57" quat="1 0 0 0">
+				<geom type="box" size="0.005 0.2425 0.0675" pos="-0.2575 0 0.0675" quat="1 0 0 0" />
+				<geom type="box" size="0.005 0.2425 0.0675" pos="0.2575 0 0.0675" quat="1 0 0 0" />
+				<geom type="box" size="0.2575 0.005 0.0675" pos="0 -0.2375 0.0675" quat="1 0 0 0" />
+				<geom type="box" size="0.2575 0.005 0.0675" pos="0 0.2375 0.0675" quat="1 0 0 0" />
+				<geom type="box" size="0.2575 0.2425 0.005" pos="0 0 0.005" quat="1 0 0 0" />
+				<joint type="slide" axis="0 1 0" range="0 0.52" />
+			</body>
+			<geom type="box" size="0.3 0.295 0.0425" pos="0 0 0.0425" quat="1 0 0 0" />
+			<geom type="box" size="0.3 0.01 0.42" pos="0 -0.285 0.42" quat="1 0 0 0" />
+			<geom type="box" size="0.01 0.27 0.42" pos="0.29 -0.025 0.42" quat="1 0 0 0" />
+			<geom type="box" size="0.01 0.27 0.42" pos="-0.29 -0.025 0.42" quat="1 0 0 0" />
+			<geom type="box" size="0.3 0.295 0.015" pos="0 0 0.825" quat="1 0 0 0" />
+		</body>
+		<body name="dining_table" pos="9.64711856842041 0.36319079995155334 0"
+			quat="-0.2098684489713483 1.583989073518146e-10 1.2484903954687643e-08 0.977729632427268">
+			<geom type="box" size="0.085 0.085 0.3575" pos="0 0 0.3575" quat="1 0 0 0" />
+			<geom type="box" size="0.3425 0.3425 0.01" pos="0 0 0.715" quat="1 0 0 0" />
+		</body>
+		<body name="desk" pos="3.0995519161224365 -1.323012113571167 0"
+			quat="-0.34838101187286763 -2.1272931977855596e-10 2.0546657661071087e-08 0.9373530127793032">
+			<geom type="box" size="0.06 0.06 0.36" pos="-0.35 -0.7005 0.36" quat="1 0 0 0" />
+			<geom type="box" size="0.06 0.06 0.36" pos="0.35 -0.7005 0.36" quat="1 0 0 0" />
+			<geom type="box" size="0.06 0.06 0.36" pos="-0.35 0.7005 0.36" quat="1 0 0 0" />
+			<geom type="box" size="0.06 0.06 0.36" pos="0.35 0.7005 0.36" quat="1 0 0 0" />
+			<geom type="box" size="0.4 0.8 0.0125" pos="0 0 0.7175" quat="1 0 0 0" />
+		</body>
+		<body name="couch_table" pos="8.048605918884277 5.848633766174316 0"
+			quat="1.9470718377062835e-07 0 0 0.9999999999999811">
 			<geom type="cylinder" size="0.2 0.005" pos="0 0 0.005" quat="1 0 0 0" />
-			<geom type="cylinder" size="0.1 0.35" pos="0 0 0.35" quat="1 0 0 0" />
-			<geom type="cylinder" size="0.45 0.0125" pos="0 0 0.715" quat="1 0 0 0" />
-		</body>
-		<body name="kitchen_refrigerator" pos="0.5147291421890259 2.1027204990386963 0"
-			quat="0.7087796582720486 -4.209975452781328e-08 -4.820778542349932e-10 0.7054299370027872">
-			<geom type="box" size="0.575 0.2965 0.4585" pos="0 0 0.4585" quat="1 0 0 0" />
-			<geom type="box" size="0.31 0.2965 1.15" pos="-0.885 0 1.15" quat="1 0 0 0" />
-		</body>
-		<body name="kitchen_oven" pos="1.8971235752105713 2.9880576133728027 0"
-			quat="0.7067220776251374 -4.23086808185462e-08 -7.055409004011468e-10 0.7074912755626089">
-			<geom type="box" size="0.315 1.569 0.6" pos="0 0 2.032" quat="1 0 0 0" />
-			<geom type="box" size="0.315 1.569 0.4585" pos="0 0 0.4585" quat="1 0 0 0" />
-		</body>
-		<body name="kitchen_counter"
-			pos="3.140516996383667 2.2580442428588867 3.725290298461914e-08"
-			quat="0.7087796582720486 -4.209975452781328e-08 -4.820812959262025e-10 0.7054299370027872">
-			<geom type="box" size="0.4 0.32 0.4585" pos="0 0 0.4585" quat="1 0 0 0" />
-		</body>
-		<body name="glass_table" pos="6.2535481452941895 1.7018171548843384 3.7159770727157593e-07"
-			quat="0.709219966328421 -2.1846834656069532e-10 -4.1716832911847685e-08 -0.7049872618431567">
-			<geom type="box" size="0.06 0.06 0.36" pos="-0.305 -0.5005 0.36" quat="1 0 0 0" />
-			<geom type="box" size="0.06 0.06 0.36" pos="0.305 -0.5005 0.36" quat="1 0 0 0" />
-			<geom type="box" size="0.06 0.06 0.36" pos="-0.305 0.5005 0.36" quat="1 0 0 0" />
-			<geom type="box" size="0.06 0.06 0.36" pos="0.305 0.5005 0.36" quat="1 0 0 0" />
-			<geom type="box" size="0.365 0.5605 0.011" pos="0 0 0.731" quat="1 0 0 0" />
-		</body>
-		<body name="couch_table" pos="6.938351631164551 -2.3634183406829834 0"
-			quat="0.7847741881010395 -8.564504703302683e-09 6.340631939708683e-10 -0.6197817952234111">
-			<geom type="box" size="0.025 0.025 0.2" pos="-0.25 -0.25 0.2" quat="1 0 0 0" />
-			<geom type="box" size="0.025 0.025 0.2" pos="0.25 -0.25 0.2" quat="1 0 0 0" />
-			<geom type="box" size="0.025 0.025 0.2" pos="-0.25 0.25 0.2" quat="1 0 0 0" />
-			<geom type="box" size="0.025 0.025 0.2" pos="0.25 0.25 0.2" quat="1 0 0 0" />
-			<geom type="box" size="0.275 0.275 0.025" pos="0 0 0.425" quat="1 0 0 0" />
-		</body>
-		<body name="couch" pos="8.280790328979492 -2.2168631553649902 6.044283509254456e-07"
-			quat="0.7087796582720486 -4.209975452781328e-08 -4.820594800448268e-10 0.7054299370027872">
-			<geom type="box" size="1 0.45 0.41" pos="0 0 0.41" quat="1 0 0 0" />
+			<geom type="cylinder" size="0.1 0.26" pos="0 0 0.26" quat="1 0 0 0" />
+			<geom type="cylinder" size="0.4 0.01" pos="0 0 0.53" quat="1 0 0 0" />
+		</body>
+		<body name="coat_hanger" pos="10.061262130737305 7.823883533477783 0"
+			quat="1.9470718377062835e-07 0 0 0.9999999999999811">
+			<geom type="cylinder" size="0.225 0.85" pos="0 0 0.85" quat="1 0 0 0" />
+		</body>
+		<body name="cabinet" pos="3.3436827659606934 1.5821243524551392 0"
+			quat="-0.023799261048375854 -3.435410285265514e-11 1.4772006932456075e-09 0.9997167574736113">
+			<geom type="box" size="0.38 0.1325 0.01" pos="0 0.007500000000000007 2.007"
+				quat="1 0 0 0" />
+			<geom type="box" size="0.38 0.1325 0.01" pos="0 0.007500000000000007 1.429"
+				quat="1 0 0 0" />
+			<geom type="box" size="0.38 0.1325 0.01" pos="0 0.007500000000000007 1.049"
+				quat="1 0 0 0" />
+			<geom type="box" size="0.38 0.1325 0.01" pos="0 0.007500000000000007 0.759"
+				quat="1 0 0 0" />
+			<geom type="box" size="0.38 0.1325 0.01"
+				pos="0 0.007500000000000007 0.44000000000000006" quat="1 0 0 0" />
+			<geom type="box" size="0.38 0.1325 0.01"
+				pos="0 0.007500000000000007 0.09000000000000001" quat="1 0 0 0" />
+			<geom type="box" size="0.38 0.007500000000000007 1.01" pos="0 -0.1325 1.01"
+				quat="1 0 0 0" />
+			<geom type="box" size="0.01 0.14 1.01" pos="0.39 0 1.01" quat="1 0 0 0" />
+			<geom type="box" size="0.01 0.14 1.01" pos="-0.39 0 1.01" quat="1 0 0 0" />
+		</body>
+		<body name="bed" pos="1.7459826469421387 5.820728778839111 4.76837158203125e-07"
+			quat="-0.025032011954692995 2.680273598670238e-10 1.7658886486176809e-09 0.9996866500946685">
+			<geom type="box" size="0.035 0.51 0.325" pos="1.035 0 0.325" quat="1 0 0 0" />
+			<geom type="box" size="0.035 0.51 0.325" pos="-1.035 0 0.325" quat="1 0 0 0" />
+			<geom type="box" size="1 0.51 0.24" pos="0 0 0.24" quat="1 0 0 0" />
+		</body>
+		<body name="bar" pos="9.598333358764648 2.5869030952453613 3.725290298461914e-09"
+			quat="-0.022114964028054965 -2.206501491923298e-10 1.4841266987394807e-09 0.9997554342768225">
+			<geom type="box" size="0.25 0.25 0.25" pos="0 0 0.25" quat="1 0 0 0" />
+		</body>
+		<body name="arm_chair" pos="10.000221252441406 3.2475147247314453 3.725290298461914e-09"
+			quat="-0.33732443731400064 5.511213515940126e-11 2.0109668407987775e-08 0.9413884554161436">
+			<geom type="box" size="0.24 0.025 0.25" pos="0 0.275 0.62" quat="1 0 0 0" />
+			<geom type="box" size="0.025 0.275 0.1" pos="0.25 0 0.47" quat="1 0 0 0" />
+			<geom type="box" size="0.025 0.275 0.1" pos="-0.25 0 0.47" quat="1 0 0 0" />
+			<geom type="box" size="0.24 0.275 0.185" pos="0 0 0.175" quat="1 0 0 0" />
 		</body>
 	</worldbody>
